File: lm35.sch (KiCad schematic (older format))
At the start: 3 parts, among them J7 Conn_01x03

Commit message: Closes #17
Changed lines of the file:
@@
 AR Path="/612F4D6E/61313C16" Ref="J7"  Part="1"
 AR Path="/61323238/61313C16" Ref="J8"  Part="1"
-F 0 "J7" H 4800 3200 50  0000 L CNN
+F 0 "J8" H 4800 3200 50  0000 L CNN
 F 1 "Conn_01x03" H 4930 2901 50  0001 L CNN
 F 2 "Connector_Molex:Molex_KK-254_AE-6410-03A_1x03_P2.54mm_Vertical" H 4850 2950 50  0001 C CNN
@@
 AR Path="/612F4D6E/61316DCA" Ref="C18"  Part="1"
 AR Path="/61323238/61316DCA" Ref="C20"  Part="1"
-F 0 "C18" H 5465 3246 50  0000 L CNN
+F 0 "C20" H 5465 3246 50  0000 L CNN
 F 1 "100nF" H 5465 3155 50  0000 L CNN
 F 2 "Capacitor_SMD:C_1206_3216Metric_Pad1.33x1.80mm_HandSolder" H 5388 3050 50  0001 C CNN
@@
 AR Path="/612F4D6E/613172FB" Ref="C19"  Part="1"
 AR Path="/61323238/613172FB" Ref="C21"  Part="1"
-F 0 "C19" H 5965 3246 50  0000 L CNN
+F 0 "C21" H 5965 3246 50  0000 L CNN
 F 1 "100nF" H 5965 3155 50  0000 L CNN
 F 2 "Capacitor_SMD:C_1206_3216Metric_Pad1.33x1.80mm_HandSolder" H 5888 3050 50  0001 C CNN
