File: mosfet-out.sch (KiCad schematic (older format))
At the start: 5 parts, among them J9 Conn_01x03, Q6 BC817, Q7 IRF540N

Commit message: Closes #14
Parts:
- removed J9: Conn_01x03, Connector_Molex:Molex_KK-254_AE-6410-03A_1x03_P2.54mm_Vertical, symbol Connector_Generic:Conn_01x03
Connections:
- net OUT: now reaches Q7.2 (D)
- no-connect marks 1 -> 0
Changed lines of the file:
@@
-	1    0    0    -1
-$EndComp
-$Comp
-L power:+12V #PWR?
-U 1 1 6138E9D9
-P 6250 2900
-AR Path="/6138E9D9" Ref="#PWR?"  Part="1"
-AR Path="/6137CC2E/6138E9D9" Ref="#PWR0147"  Part="1"
-F 0 "#PWR0147" H 6250 2750 50  0001 C CNN
-F 1 "+12V" H 6265 3073 50  0000 C CNN
-F 2 "" H 6250 2900 50  0001 C CNN
-F 3 "" H 6250 2900 50  0001 C CNN
-	1    6250 2900
 	1    0    0    -1
 $EndComp
@@
 	5850 3000 5850 2900
 Wire Wire Line
-	6250 2900 6250 2950
-Wire Wire Line
-	6250 2950 6450 2950
-Wire Wire Line
 	6450 3150 6250 3150
 Wire Wire Line
@@
 Wire Wire Line
 	6250 3950 6250 3600
-NoConn ~ 6450 3050
-$Comp
-L Connector_Generic:Conn_01x03 J?
-U 1 1 6138E9EA
-P 6650 3050
-AR Path="/6138E9EA" Ref="J?"  Part="1"
-AR Path="/6137CC2E/6138E9EA" Ref="J9"  Part="1"
-F 0 "J9" H 6500 3300 50  0000 L CNN
-F 1 "Conn_01x03" H 6730 3001 50  0001 L CNN
-F 2 "Connector_Molex:Molex_KK-254_AE-6410-03A_1x03_P2.54mm_Vertical" H 6650 3050 50  0001 C CNN
-F 3 "https://app.adam-tech.com/products/download/data_sheet/196588/lha-xx-ts-data-sheet.pdf" H 6650 3050 50  0001 C CNN
-F 4 "LHA-03-TS" H 6650 3050 50  0001 C CNN "manf#"
-	1    6650 3050
-	1    0    0    -1
-$EndComp
 Text HLabel 4900 3700 0    39   Input ~ 0
 ON
 Wire Wire Line
 	4900 3700 5200 3700
+Text HLabel 6450 3150 2    39   Output ~ 0
+OUT
 $EndSCHEMATC

Commit message: Several changes
Usando stock de http://tienda.ityt.com.ar/
Parts:
- removed Q7: IRF540N, Package_TO_SOT_THT:TO-220-3_Vertical, symbol Transistor_FET:IRF540N
- added Q7: IRLML2502, Package_TO_SOT_SMD:SOT-23, symbol Transistor_FET:IRLML0030
Connections:
- net GND: now also Q7.2 (S)
- net OUT: now also Q7.3 (D)
- net at Q6.3 (C), R28.2: now also Q7.1 (G)
Changed lines of the file:
@@
 $Descr A4 11693 8268
 encoding utf-8
-Sheet 14 19
+Sheet 14 18
 Title "12V Power Output"
 Date "2021-06-10"
@@
 Comment4 ""
 $EndDescr
-$Comp
-L Transistor_FET:IRF540N Q?
-U 1 1 6138E9AB
-P 6150 3400
-AR Path="/6138E9AB" Ref="Q?"  Part="1"
-AR Path="/6137CC2E/6138E9AB" Ref="Q7"  Part="1"
-F 0 "Q7" H 6354 3446 50  0000 L CNN
-F 1 "IRF540N" H 6354 3355 50  0000 L CNN
-F 2 "Package_TO_SOT_THT:TO-220-3_Vertical" H 6400 3325 50  0001 L CIN
-F 3 "https://www.infineon.com/dgdl/irf540nspbf.pdf?fileId=5546d462533600a4015355e3a72819a3" H 6150 3400 50  0001 L CNN
-F 4 "IRF540NLPBF" H 6150 3400 50  0001 C CNN "manf#"
-	1    6150 3400
-	1    0    0    -1
-$EndComp
 $Comp
 L power:GND #PWR?
@@
 Text HLabel 6450 3150 2    39   Output ~ 0
 OUT
+$Comp
+L Transistor_FET:IRLML0030 Q7
+U 1 1 60DD41B1
+P 6150 3400
+F 0 "Q7" H 6354 3446 50  0000 L CNN
+F 1 "IRLML2502" H 6354 3355 50  0000 L CNN
+F 2 "Package_TO_SOT_SMD:SOT-23" H 6350 3325 50  0001 L CIN
+F 3 "https://www.infineon.com/dgdl/irlml2502pbf.pdf?fileId=5546d462533600a401535668048e2606" H 6150 3400 50  0001 L CNN
+F 4 "IRLML2502TRPBF" H 6150 3400 50  0001 C CNN "manf#"
+	1    6150 3400
+	1    0    0    -1
+$EndComp
 $EndSCHEMATC
