File: serialport.sch (KiCad schematic (older format))
At the start: 11 parts, among them J6 USB_B, Q4 BC817, Q5 BC817, U1 CH340G, Y1 12MHz

Commit message: new footprints
Parts:
- J6: footprint Connector_USB:USB_B_TE_5787834_Vertical -> libs:USB-B-VERTICAL-SMD&THT
Changed lines of the file:
@@
 F 0 "J6" H 3857 3817 50  0000 C CNN
 F 1 "USB_B" H 3857 3726 50  0000 C CNN
-F 2 "Connector_USB:USB_B_TE_5787834_Vertical" H 3950 3300 50  0001 C CNN
+F 2 "libs:USB-B-VERTICAL-SMD&THT" H 3950 3300 50  0001 C CNN
 F 3 "https://www.te.com/commerce/DocumentDelivery/DDEController?Action=srchrtrv&DocNm=5787834&DocType=Customer+Drawing&DocLang=English" H 3950 3300 50  0001 C CNN
 F 4 "5787834-1" H 3800 3350 50  0001 C CNN "manf#"

Commit message: Closes #17
Parts:
- added J11: ICSP, Connector_PinSocket_2.54mm:PinSocket_1x06_P2.54mm_Vertical, symbol Connector_Generic:Conn_01x06
Connections:
- net +3V3: now also J11.6 (Pin_6)
- net FLASH_uC: now also J11.4 (Pin_4)
- net GND: now also J11.5 (Pin_5)
- net RESET_uC: now also J11.1 (Pin_1)
- net RXD: now also J11.2 (Pin_2)
- net TXD: now also J11.3 (Pin_3)
Other:
- moved on the sheet: C13, C2, C3, C4, J6, Q4, Q5, R13, R14, U1, Y1
