File: currentsensor.sch (KiCad schematic (older format))
At the start: 9 parts, among them U2 ACS759, U3 ACS712

Commit message: more footprints & 3d models
Parts:
- U2: footprint Sensor_Current:Allegro_CB_PFF -> libs:Allegro_CB_PFF
Changed lines of the file:
@@
 F 0 "U2" H 6600 5150 50  0000 L CNN
 F 1 "ACS759" H 5450 4600 50  0000 L CNN
-F 2 "Sensor_Current:Allegro_CB_PFF" H 6400 4900 50  0001 C CNN
+F 2 "libs:Allegro_CB_PFF" H 6400 4900 50  0001 C CNN
 F 3 "https://www.allegromicro.com/~/media/Files/Datasheets/ACS759-Datasheet.ashx" H 6400 4900 50  0001 C CNN
 F 4 "ACS759LCB-050B-PFF-T" H 6400 4900 50  0001 C CNN "manf#"
