File: kicad.sch (KiCad schematic (older format))
At the start: 46 parts, among them J1 Screw_Terminal_01x03, J2 Conn_01x06, J3 Screw_Terminal_01x03, J4 Conn_01x03, J5 Conn_01x03, J6 Conn_01x03, J7 Conn_01x04, J8 Screw_Terminal_01x02, K1 SANYOU_SRD_Form_C, K2 SANYOU_SRD_Form_C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

Commit message: Several changes.
Parts:
- removed C2, C3, C4: 100nF, Capacitor_SMD:C_1206_3216Metric_Pad1.33x1.80mm_HandSolder, symbol Device:C
- removed D1, D2, D3: 1N4007, Diode_THT:D_DO-41_SOD81_P7.62mm_Horizontal, symbol Diode:1N4007
- removed D?: LED, symbol Device:LED
- removed J1: Screw_Terminal_01x03, TerminalBlock:TerminalBlock_bornier-3_P5.08mm, symbol Connector:Screw_Terminal_01x03
- removed J2: Conn_01x06, symbol Connector_Generic:Conn_01x06
- removed J4, J5, J6: Conn_01x03, symbol Connector_Generic:Conn_01x03
- removed J7: Conn_01x04, symbol Connector_Generic:Conn_01x04
- removed K1, K2: SANYOU_SRD_Form_C, Relay_THT:Relay_SPDT_SANYOU_SRD_Series_Form_C, symbol Relay:SANYOU_SRD_Form_C
- removed Q1, Q2, Q3, Q4: BC817, Package_TO_SOT_SMD:SOT-23, symbol Transistor_BJT:BC817
- removed Q5: IRF540N, Package_TO_SOT_THT:TO-220-3_Vertical, symbol Transistor_FET:IRF540N
- removed R10, R7, R8: 1k, Resistor_SMD:R_1206_3216Metric_Pad1.30x1.75mm_HandSolder, symbol Device:R
- removed R3, R4, R5, R6, R9: 10k, Resistor_SMD:R_1206_3216Metric_Pad1.30x1.75mm_HandSolder, symbol Device:R
- removed R?: 1k, symbol Device:R
- removed U1, U2, U3, U4: 4N25, Package_DIP:DIP-6_W7.62mm, symbol Isolator:4N25
- removed U5: ACS759xCB-050B-PFF, Sensor_Current:Allegro_CB_PFF, symbol Sensor_Current:ACS759xCB-050B-PFF
- added D1, D2: SS14, Diode_SMD:D_SMA, symbol Diode:B140-E3
- added D3, D4: ALT, Diode_SMD:D_SMA, symbol Diode:B140-E3
- added J2, J5: Screw_Terminal_01x03, TerminalBlock:TerminalBlock_bornier-3_P5.08mm, symbol Connector:Screw_Terminal_01x03
- added J4: Conn_01x05, symbol Connector_Generic:Conn_01x05
- added SW1, SW2: SW_Push, symbol Switch:SW_Push
- R1, R2: value 1k -> 10K
- U6: renamed from U?; value ESP32-WROOM-32 -> ESP32
- renumbered J8 to J1, R13 to R5, R14 to R6
Connections:
- net labels added: +5V, GPIO0, RELAY_3, RESET, RXD0, TXD0, VUSB
- wire segments 190 -> 107
- no-connect marks 25 -> 16
Other:
- note added: "*Optional."
- note added: "12v SWITCHED OUTPUT"
- note added: "PUSHBUTTONS"
- note added: "TEMPERATURE SENSORS"
- note added: "UPS-INTERFACE"
- note added: "USB Power"
- note removed: "BATT. TEMP."
- note removed: "COOLER OUTPUT"
- note removed: "EXTRA_TEMP"
- note removed: "UPS INTERFACE"
- moved on the sheet: J1, R11, R12, R5, R6, U6

Commit message: updated all components
Parts:
- C1: Voltage (none) -> 50V; manf# (none) -> CC1206KRX7R9BB104
- D1, D2: footprint Diode_SMD:D_SMA -> Diode_SMD:D_SMA_Handsoldering; manf# (none) -> SS14
- D3, D4: footprint Diode_SMD:D_SMA -> Diode_THT:D_DO-201_P12.70mm_Horizontal; manf# (none) -> 1N5819
- J1: manf# (none) -> 796636-2
- J2, J3, J5: manf# (none) -> 796636-3
- J4: footprint (none) -> Connector_Molex:Molex_KK-254_AE-6410-05A_1x05_P2.54mm_Vertical; manf# (none) -> LHA-05-TS
- R1, R11, R12, R2: value 10K -> 10k; footprint Resistor_SMD:R_1206_3216Metric_Pad1.30x1.75mm_HandSolder -> Resistor_SMD:R_1206_3216Metric; manf# (none) -> RC1206FR-0710KL
- R5: footprint Resistor_SMD:R_0805_2012Metric_Pad1.20x1.40mm_HandSolder -> Resistor_SMD:R_1206_3216Metric; manf# (none) -> RC1206FR-0722KL
- R6: footprint Resistor_SMD:R_0805_2012Metric_Pad1.20x1.40mm_HandSolder -> Resistor_SMD:R_1206_3216Metric; manf# (none) -> RC1206FR-075K6L
- SW1, SW2: footprint (none) -> Button_Switch_THT:SW_PUSH_6mm; manf# (none) -> 1-1825910-0
- U6: manf# (none) -> ESP32-WROOM-32E
Changed lines of the file:
@@
 P 4400 6750
 F 0 "R12" H 4470 6796 50  0000 L CNN
-F 1 "10K" H 4470 6705 50  0000 L CNN
-F 2 "Resistor_SMD:R_1206_3216Metric_Pad1.30x1.75mm_HandSolder" V 4330 6750 50  0001 C CNN
-F 3 "~" H 4400 6750 50  0001 C CNN
+F 1 "10k" H 4470 6705 50  0000 L CNN
+F 2 "Resistor_SMD:R_1206_3216Metric" V 4330 6750 50  0001 C CNN
+F 3 "https://www.yageo.com/upload/media/product/productsearch/datasheet/rchip/PYu-RC_Group_51_RoHS_L_11.pdf" H 4400 6750 50  0001 C CNN
+F 4 "RC1206FR-0710KL" H 4400 6750 50  0001 C CNN "manf#"
 	1    4400 6750
 	1    0    0    -1
@@
 P 4100 6750
 F 0 "R11" H 4170 6796 50  0000 L CNN
-F 1 "10K" H 4170 6705 50  0000 L CNN
-F 2 "Resistor_SMD:R_1206_3216Metric_Pad1.30x1.75mm_HandSolder" V 4030 6750 50  0001 C CNN
-F 3 "~" H 4100 6750 50  0001 C CNN
+F 1 "10k" H 4170 6705 50  0000 L CNN
+F 2 "Resistor_SMD:R_1206_3216Metric" V 4030 6750 50  0001 C CNN
+F 3 "https://www.yageo.com/upload/media/product/productsearch/datasheet/rchip/PYu-RC_Group_51_RoHS_L_11.pdf" H 4100 6750 50  0001 C CNN
+F 4 "RC1206FR-0710KL" H 4100 6750 50  0001 C CNN "manf#"
 	1    4100 6750
 	1    0    0    -1
@@
 F 0 "R5" H 1770 6896 50  0000 L CNN
 F 1 "22k" H 1770 6805 50  0000 L CNN
-F 2 "Resistor_SMD:R_0805_2012Metric_Pad1.20x1.40mm_HandSolder" V 1630 6850 50  0001 C CNN
-F 3 "~" H 1700 6850 50  0001 C CNN
+F 2 "Resistor_SMD:R_1206_3216Metric" V 1630 6850 50  0001 C CNN
+F 3 "https://www.yageo.com/upload/media/product/productsearch/datasheet/rchip/PYu-RC_Group_51_RoHS_L_11.pdf" H 1700 6850 50  0001 C CNN
+F 4 "RC1206FR-0722KL" H 1700 6850 50  0001 C CNN "manf#"
 	1    1700 6850
 	1    0    0    -1
@@
 F 0 "R6" H 1770 7296 50  0000 L CNN
 F 1 "5k6" H 1770 7205 50  0000 L CNN
-F 2 "Resistor_SMD:R_0805_2012Metric_Pad1.20x1.40mm_HandSolder" V 1630 7250 50  0001 C CNN
-F 3 "~" H 1700 7250 50  0001 C CNN
+F 2 "Resistor_SMD:R_1206_3216Metric" V 1630 7250 50  0001 C CNN
+F 3 "https://www.yageo.com/upload/media/product/productsearch/datasheet/rchip/PYu-RC_Group_51_RoHS_L_11.pdf" H 1700 7250 50  0001 C CNN
+F 4 "RC1206FR-075K6L" H 1700 7250 50  0001 C CNN "manf#"
 	1    1700 7250
 	1    0    0    -1
@@
 F 1 "Screw_Terminal_01x02" H 618 6776 50  0001 C CNN
 F 2 "TerminalBlock:TerminalBlock_bornier-2_P5.08mm" H 700 6650 50  0001 C CNN
-F 3 "~" H 700 6650 50  0001 C CNN
+F 3 "https://www.te.com/commerce/DocumentDelivery/DDEController?Action=srchrtrv&DocNm=796636&DocType=Customer+Drawing&DocLang=English" H 700 6650 50  0001 C CNN
+F 4 "796636-2" H 700 6650 50  0001 C CNN "manf#"
 	1    700  6650
 	-1   0    0    -1
@@
 F 0 "D2" H 1400 6750 50  0000 C CNN
 F 1 "SS14" H 1200 6750 50  0000 C CNN
-F 2 "Diode_SMD:D_SMA" H 1300 6475 50  0001 C CNN
-F 3 "https://www.vishay.com/docs/88746/ss12.pdf" H 1300 6650 50  0001 C CNN
+F 2 "Diode_SMD:D_SMA_Handsoldering" H 1300 6475 50  0001 C CNN
+F 3 "https://www.onsemi.com/pdf/datasheet/ss19-d.pdf" H 1300 6650 50  0001 C CNN
+F 4 "SS14" H 1300 6650 50  0001 C CNN "manf#"
 	1    1300 6650
 	-1   0    0    -1
@@
 F 0 "D3" H 1400 6950 50  0000 C CNN
 F 1 "ALT" H 1200 6950 50  0000 C CNN
-F 2 "Diode_SMD:D_SMA" H 1300 6675 50  0001 C CNN
-F 3 "https://www.vishay.com/docs/88746/ss12.pdf" H 1300 6850 50  0001 C CNN
+F 2 "Diode_THT:D_DO-201_P12.70mm_Horizontal" H 1300 6675 50  0001 C CNN
+F 3 "https://www.st.com/content/ccc/resource/technical/document/datasheet/26/db/14/60/52/47/47/5b/CD00001625.pdf/files/CD00001625.pdf/jcr:content/translations/en.CD00001625.pdf" H 1300 6850 50  0001 C CNN
+F 4 "1N5819" H 1300 6850 50  0001 C CNN "manf#"
 	1    1300 6850
 	-1   0    0    -1
@@
 F 0 "J4" H 4950 7500 50  0000 L CNN
 F 1 "Conn_01x05" H 5180 7101 50  0001 L CNN
-F 2 "" H 5100 7150 50  0001 C CNN
-F 3 "~" H 5100 7150 50  0001 C CNN
+F 2 "Connector_Molex:Molex_KK-254_AE-6410-05A_1x05_P2.54mm_Vertical" H 5100 7150 50  0001 C CNN
+F 3 "https://app.adam-tech.com/products/download/data_sheet/196588/lha-xx-ts-data-sheet.pdf" H 5100 7150 50  0001 C CNN
+F 4 "LHA-05-TS" H 5100 7150 50  0001 C CNN "manf#"
 	1    5100 7150
 	1    0    0    -1
@@
 F 1 "ESP32" H 9350 4800 50  0000 C CNN
 F 2 "RF_Module:ESP32-WROOM-32" H 9700 1950 50  0001 C CNN
-F 3 "https://www.espressif.com/sites/default/files/documentation/esp32-wroom-32_datasheet_en.pdf" H 9400 3500 50  0001 C CNN
+F 3 "https://www.espressif.com/sites/default/files/documentation/esp32-wroom-32e_esp32-wroom-32ue_datasheet_en.pdf" H 9400 3500 50  0001 C CNN
+F 4 "ESP32-WROOM-32E" H 9700 3450 50  0001 C CNN "manf#"
 	1    9700 3450
 	-1   0    0    -1
@@
 F 1 "100nF" H 10665 3055 50  0000 L CNN
 F 2 "Capacitor_SMD:C_1206_3216Metric_Pad1.33x1.80mm_HandSolder" H 10588 2950 50  0001 C CNN
-F 3 "~" H 10550 3100 50  0001 C CNN
+F 3 "https://www.yageo.com/upload/media/product/productsearch/datasheet/mlcc/UPY-GPHC_X7R_6.3V-to-50V_18.pdf" H 10550 3100 50  0001 C CNN
+F 4 "50V" H 10550 3100 50  0001 C CNN "Voltage"
+F 5 "CC1206KRX7R9BB104" H 10550 3100 50  0001 C CNN "manf#"
 	1    10550 3100
 	1    0    0    -1
@@
 F 0 "D1" H 1400 7450 50  0000 C CNN
 F 1 "SS14" H 1200 7450 50  0000 C CNN
-F 2 "Diode_SMD:D_SMA" H 1300 7175 50  0001 C CNN
-F 3 "https://www.vishay.com/docs/88746/ss12.pdf" H 1300 7350 50  0001 C CNN
+F 2 "Diode_SMD:D_SMA_Handsoldering" H 1300 7175 50  0001 C CNN
+F 3 "https://www.onsemi.com/pdf/datasheet/ss19-d.pdf" H 1300 7350 50  0001 C CNN
 F 4 "No" H 1300 7350 50  0001 C CNN "Fixed"
+F 5 "SS14" H 1300 7350 50  0001 C CNN "manf#"
 	1    1300 7350
 	-1   0    0    -1
@@
 F 0 "D4" H 1400 7650 50  0000 C CNN
 F 1 "ALT" H 1200 7650 50  0000 C CNN
-F 2 "Diode_SMD:D_SMA" H 1300 7375 50  0001 C CNN
-F 3 "https://www.vishay.com/docs/88746/ss12.pdf" H 1300 7550 50  0001 C CNN
+F 2 "Diode_THT:D_DO-201_P12.70mm_Horizontal" H 1300 7375 50  0001 C CNN
+F 3 "https://www.st.com/content/ccc/resource/technical/document/datasheet/26/db/14/60/52/47/47/5b/CD00001625.pdf/files/CD00001625.pdf/jcr:content/translations/en.CD00001625.pdf" H 1300 7550 50  0001 C CNN
 F 4 "No" H 1300 7550 50  0001 C CNN "Fixed"
+F 5 "1N5819" H 1300 7550 50  0001 C CNN "manf#"
 	1    1300 7550
 	-1   0    0    -1
@@
 F 1 "Screw_Terminal_01x03" H 2030 4601 50  0001 L CNN
 F 2 "TerminalBlock:TerminalBlock_bornier-3_P5.08mm" H 1950 4650 50  0001 C CNN
-F 3 "~" H 1950 4650 50  0001 C CNN
+F 3 "https://www.te.com/commerce/DocumentDelivery/DDEController?Action=srchrtrv&DocNm=796636&DocType=Customer+Drawing&DocLang=English" H 1950 4650 50  0001 C CNN
+F 4 "796636-3" H 1950 4650 50  0001 C CNN "manf#"
 	1    1950 4650
 	1    0    0    -1
@@
 F 1 "Screw_Terminal_01x03" H 2030 5201 50  0001 L CNN
 F 2 "TerminalBlock:TerminalBlock_bornier-3_P5.08mm" H 1950 5250 50  0001 C CNN
-F 3 "~" H 1950 5250 50  0001 C CNN
+F 3 "https://www.te.com/commerce/DocumentDelivery/DDEController?Action=srchrtrv&DocNm=796636&DocType=Customer+Drawing&DocLang=English" H 1950 5250 50  0001 C CNN
+F 4 "796636-3" H 1950 5250 50  0001 C CNN "manf#"
 	1    1950 5250
 	1    0    0    -1
@@
 F 1 "Screw_Terminal_01x03" H 2030 5801 50  0001 L CNN
 F 2 "TerminalBlock:TerminalBlock_bornier-3_P5.08mm" H 1950 5850 50  0001 C CNN
-F 3 "~" H 1950 5850 50  0001 C CNN
+F 3 "https://www.te.com/commerce/DocumentDelivery/DDEController?Action=srchrtrv&DocNm=796636&DocType=Customer+Drawing&DocLang=English" H 1950 5850 50  0001 C CNN
+F 4 "796636-3" H 1950 5850 50  0001 C CNN "manf#"
 	1    1950 5850
 	1    0    0    -1
@@
 F 0 "SW2" H 2800 6000 50  0000 C CNN
 F 1 "SW_Push" H 2650 6094 50  0001 C CNN
-F 2 "" H 2650 6100 50  0001 C CNN
-F 3 "~" H 2650 6100 50  0001 C CNN
+F 2 "Button_Switch_THT:SW_PUSH_6mm" H 2650 6100 50  0001 C CNN
+F 3 "https://www.te.com/commerce/DocumentDelivery/DDEController?Action=srchrtrv&DocNm=1825910&DocType=Customer+Drawing&DocLang=English" H 2650 6100 50  0001 C CNN
+F 4 "1-1825910-0" H 2650 5900 50  0001 C CNN "manf#"
 	1    2650 5900
 	1    0    0    -1
@@
 F 0 "SW1" H 2800 5750 50  0000 C CNN
 F 1 "SW_Push" H 2650 5844 50  0001 C CNN
-F 2 "" H 2650 5850 50  0001 C CNN
-F 3 "~" H 2650 5850 50  0001 C CNN
+F 2 "Button_Switch_THT:SW_PUSH_6mm" H 2650 5850 50  0001 C CNN
+F 3 "https://www.te.com/commerce/DocumentDelivery/DDEController?Action=srchrtrv&DocNm=1825910&DocType=Customer+Drawing&DocLang=English" H 2650 5850 50  0001 C CNN
+F 4 "1-1825910-0" H 2650 5650 50  0001 C CNN "manf#"
 	1    2650 5650
 	1    0    0    -1
@@
 P 2950 5400
 F 0 "R1" H 3020 5446 50  0000 L CNN
-F 1 "10K" H 3020 5355 50  0000 L CNN
-F 2 "Resistor_SMD:R_1206_3216Metric_Pad1.30x1.75mm_HandSolder" V 2880 5400 50  0001 C CNN
-F 3 "~" H 2950 5400 50  0001 C CNN
+F 1 "10k" H 3020 5355 50  0000 L CNN
+F 2 "Resistor_SMD:R_1206_3216Metric" V 2880 5400 50  0001 C CNN
+F 3 "https://www.yageo.com/upload/media/product/productsearch/datasheet/rchip/PYu-RC_Group_51_RoHS_L_11.pdf" H 2950 5400 50  0001 C CNN
+F 4 "RC1206FR-0710KL" H 2950 5400 50  0001 C CNN "manf#"
 	1    2950 5400
 	1    0    0    -1
@@
 P 3250 5400
 F 0 "R2" H 3320 5446 50  0000 L CNN
-F 1 "10K" H 3320 5355 50  0000 L CNN
-F 2 "Resistor_SMD:R_1206_3216Metric_Pad1.30x1.75mm_HandSolder" V 3180 5400 50  0001 C CNN
-F 3 "~" H 3250 5400 50  0001 C CNN
+F 1 "10k" H 3320 5355 50  0000 L CNN
+F 2 "Resistor_SMD:R_1206_3216Metric" V 3180 5400 50  0001 C CNN
+F 3 "https://www.yageo.com/upload/media/product/productsearch/datasheet/rchip/PYu-RC_Group_51_RoHS_L_11.pdf" H 3250 5400 50  0001 C CNN
+F 4 "RC1206FR-0710KL" H 3250 5400 50  0001 C CNN "manf#"
 	1    3250 5400
 	1    0    0    -1

Commit message: various updates
Parts:
- H1, H2: footprint (none) -> MountingHole:MountingHole_4mm_Pad_Via
Connections:
- net RELAY_3: now also U6.37 (IO23)
- no-connect marks 16 -> 15
Other:
- moved on the sheet: C1, U6
