File: relay.sch (KiCad schematic (older format))
At the start: 6 parts, among them K1 SANYOU_SRD_Form_C, Q1 BC817

Commit message: updated all components
Parts:
- D5: footprint (none) -> LED_SMD:LED_1206_3216Metric; manf# (none) -> BR1101W-TR
- D8: manf# (none) -> 1N4007G
- K1: value SANYOU_SRD_Form_C -> RELAY; manf# (none) -> G5LE-1-VDDC12
- Q1: manf# (none) -> SBC817-40LT1G
- R3: footprint (none) -> Resistor_SMD:R_1206_3216Metric; manf# (none) -> RC1206FR-071KL
- R4: footprint Resistor_SMD:R_1206_3216Metric_Pad1.30x1.75mm_HandSolder -> Resistor_SMD:R_1206_3216Metric; manf# (none) -> RC1206FR-071KL
Changed lines of the file:
@@
 F 1 "BC817" H 5641 4555 50  0000 L CNN
 F 2 "Package_TO_SOT_SMD:SOT-23" H 5650 4525 50  0001 L CIN
-F 3 "https://www.onsemi.com/pub/Collateral/BC818-D.pdf" H 5450 4600 50  0001 L CNN
+F 3 "https://www.onsemi.com/pub/Collateral/BC817-16LT1-D.PDF" H 5450 4600 50  0001 L CNN
+F 4 "SBC817-40LT1G" H 5450 4600 50  0001 C CNN "manf#"
 	1    5450 4600
 	1    0    0    -1
@@
 F 0 "R10" V 4950 4500 50  0000 C CNN
 F 1 "1k" V 4950 4700 50  0000 C CNN
-F 2 "Resistor_SMD:R_1206_3216Metric_Pad1.30x1.75mm_HandSolder" V 4980 4600 50  0001 C CNN
-F 3 "~" H 5050 4600 50  0001 C CNN
+F 2 "Resistor_SMD:R_1206_3216Metric" V 4980 4600 50  0001 C CNN
+F 3 "https://www.yageo.com/upload/media/product/productsearch/datasheet/rchip/PYu-RC_Group_51_RoHS_L_11.pdf" H 5050 4600 50  0001 C CNN
+F 4 "RC1206FR-071KL" H 5050 4600 50  0001 C CNN "manf#"
 	1    5050 4600
 	0    1    1    0
@@
 F 1 "1N4007" V 5600 3550 50  0000 L CNN
 F 2 "Diode_THT:D_DO-41_SOD81_P7.62mm_Horizontal" H 5550 3775 50  0001 C CNN
-F 3 "http://www.vishay.com/docs/88503/1n4001.pdf" H 5550 3950 50  0001 C CNN
+F 3 "https://media.digikey.com/pdf/Data%20Sheets/NextGen%20Components%20PDFs/DO41N4007GA10A.pdf" H 5550 3950 50  0001 C CNN
+F 4 "1N4007G" H 5550 3950 50  0001 C CNN "manf#"
 	1    5550 3950
 	0    1    1    0
@@
 AR Path="/610C441E/61070A63" Ref="K3"  Part="1"
 F 0 "K3" H 6000 4200 50  0000 L CNN
-F 1 "SANYOU_SRD_Form_C" H 6830 3905 50  0001 L CNN
+F 1 "RELAY" H 6830 3905 50  0001 L CNN
 F 2 "Relay_THT:Relay_SPDT_SANYOU_SRD_Series_Form_C" H 6850 3900 50  0001 L CNN
-F 3 "http://www.sanyourelay.ca/public/products/pdf/SRD.pdf" H 6400 3950 50  0001 C CNN
+F 3 "https://omronfs.omron.com/en_US/ecb/products/pdf/en-g5le.pdf" H 6400 3950 50  0001 C CNN
+F 4 "G5LE-1-VDDC12" H 6400 3950 50  0001 C CNN "manf#"
 	1    6400 3950
 	1    0    0    -1
@@
 F 0 "D12" V 4889 3632 50  0000 R CNN
 F 1 "LED" V 4798 3632 50  0000 R CNN
-F 2 "" H 4850 3750 50  0001 C CNN
-F 3 "~" H 4850 3750 50  0001 C CNN
+F 2 "LED_SMD:LED_1206_3216Metric" H 4850 3750 50  0001 C CNN
+F 3 "https://media.digikey.com/pdf/Data%20Sheets/Stanley%20Electric%20PDFs/1101W_Series.pdf" H 4850 3750 50  0001 C CNN
+F 4 "BR1101W-TR" H 4850 3750 50  0001 C CNN "manf#"
 	1    4850 3750
 	0    -1   -1   0
@@
 F 0 "R9" H 4920 4196 50  0000 L CNN
 F 1 "1k" H 4920 4105 50  0000 L CNN
-F 2 "" V 4780 4150 50  0001 C CNN
-F 3 "~" H 4850 4150 50  0001 C CNN
+F 2 "Resistor_SMD:R_1206_3216Metric" V 4780 4150 50  0001 C CNN
+F 3 "https://www.yageo.com/upload/media/product/productsearch/datasheet/rchip/PYu-RC_Group_51_RoHS_L_11.pdf" H 4850 4150 50  0001 C CNN
+F 4 "RC1206FR-071KL" H 4850 4150 50  0001 C CNN "manf#"
 	1    4850 4150
 	1    0    0    -1

Commit message: various updates
Changed lines of the file:
@@
 $Descr A4 11693 8268
 encoding utf-8
-Sheet 6 19
+Sheet 4 19
 Title ""
 Date ""
@@
 AR Path="/610A0B30/61070A3B" Ref="Q2"  Part="1"
 AR Path="/610C441E/61070A3B" Ref="Q3"  Part="1"
-F 0 "Q3" H 5641 4646 50  0000 L CNN
+F 0 "Q1" H 5641 4646 50  0000 L CNN
 F 1 "BC817" H 5641 4555 50  0000 L CNN
 F 2 "Package_TO_SOT_SMD:SOT-23" H 5650 4525 50  0001 L CIN
@@
 AR Path="/610A0B30/61070A47" Ref="R8"  Part="1"
 AR Path="/610C441E/61070A47" Ref="R10"  Part="1"
-F 0 "R10" V 4950 4500 50  0000 C CNN
+F 0 "R4" V 4950 4500 50  0000 C CNN
 F 1 "1k" V 4950 4700 50  0000 C CNN
 F 2 "Resistor_SMD:R_1206_3216Metric" V 4980 4600 50  0001 C CNN
@@
 AR Path="/610A0B30/61070A4D" Ref="D11"  Part="1"
 AR Path="/610C441E/61070A4D" Ref="D13"  Part="1"
-F 0 "D13" V 5500 3750 50  0000 L CNN
+F 0 "D8" V 5500 3750 50  0000 L CNN
 F 1 "1N4007" V 5600 3550 50  0000 L CNN
 F 2 "Diode_THT:D_DO-41_SOD81_P7.62mm_Horizontal" H 5550 3775 50  0001 C CNN
@@
 AR Path="/610A0B30/61070A63" Ref="K2"  Part="1"
 AR Path="/610C441E/61070A63" Ref="K3"  Part="1"
-F 0 "K3" H 6000 4200 50  0000 L CNN
+F 0 "K1" H 6000 4200 50  0000 L CNN
 F 1 "RELAY" H 6830 3905 50  0001 L CNN
 F 2 "Relay_THT:Relay_SPDT_SANYOU_SRD_Series_Form_C" H 6850 3900 50  0001 L CNN
@@
 Text HLabel 4650 4600 0    39   Input ~ 0
 ON
-Wire Wire Line
-	4650 4600 4900 4600
 Text HLabel 6900 3550 2    39   Output ~ 0
 NO
@@
 AR Path="/610A0B30/6107B2AB" Ref="D10"  Part="1"
 AR Path="/610C441E/6107B2AB" Ref="D12"  Part="1"
-F 0 "D12" V 4889 3632 50  0000 R CNN
+F 0 "D5" V 4889 3632 50  0000 R CNN
 F 1 "LED" V 4798 3632 50  0000 R CNN
 F 2 "LED_SMD:LED_1206_3216Metric" H 4850 3750 50  0001 C CNN
@@
 AR Path="/610A0B30/6107B2B1" Ref="R7"  Part="1"
 AR Path="/610C441E/6107B2B1" Ref="R9"  Part="1"
-F 0 "R9" H 4920 4196 50  0000 L CNN
+F 0 "R3" H 4920 4196 50  0000 L CNN
 F 1 "1k" H 4920 4105 50  0000 L CNN
 F 2 "Resistor_SMD:R_1206_3216Metric" V 4780 4150 50  0001 C CNN
@@
 Wire Wire Line
 	5550 4350 6200 4350
+Wire Wire Line
+	4650 4600 4900 4600
 $EndSCHEMATC
