File: relay.sch (KiCad schematic (older format))
At the start: 6 parts, among them K1 RELAY, Q1 BC817

Commit message: Closes #17
Changed lines of the file:
@@
 AR Path="/610A0B30/61070A3B" Ref="Q2"  Part="1"
 AR Path="/610C441E/61070A3B" Ref="Q3"  Part="1"
-F 0 "Q2" H 5641 4646 50  0000 L CNN
+F 0 "Q3" H 5641 4646 50  0000 L CNN
 F 1 "BC817" H 5641 4555 50  0000 L CNN
 F 2 "Package_TO_SOT_SMD:SOT-23" H 5650 4525 50  0001 L CIN
@@
 AR Path="/610A0B30/61070A47" Ref="R8"  Part="1"
 AR Path="/610C441E/61070A47" Ref="R10"  Part="1"
-F 0 "R8" V 4950 4500 50  0000 C CNN
+F 0 "R10" V 4950 4500 50  0000 C CNN
 F 1 "1k" V 4950 4700 50  0000 C CNN
 F 2 "Resistor_SMD:R_1206_3216Metric" V 4980 4600 50  0001 C CNN
@@
 AR Path="/610A0B30/61070A4D" Ref="D11"  Part="1"
 AR Path="/610C441E/61070A4D" Ref="D13"  Part="1"
-F 0 "D11" V 5500 3750 50  0000 L CNN
+F 0 "D13" V 5500 3750 50  0000 L CNN
 F 1 "1N4007" V 5600 3550 50  0000 L CNN
 F 2 "Diode_THT:D_DO-41_SOD81_P7.62mm_Horizontal" H 5550 3775 50  0001 C CNN
@@
 AR Path="/610A0B30/61070A63" Ref="K2"  Part="1"
 AR Path="/610C441E/61070A63" Ref="K3"  Part="1"
-F 0 "K2" H 6000 4200 50  0000 L CNN
+F 0 "K3" H 6000 4200 50  0000 L CNN
 F 1 "RELAY" H 6830 3905 50  0001 L CNN
 F 2 "Relay_THT:Relay_SPDT_SANYOU_SRD_Series_Form_C" H 6850 3900 50  0001 L CNN
@@
 AR Path="/610A0B30/6107B2AB" Ref="D10"  Part="1"
 AR Path="/610C441E/6107B2AB" Ref="D12"  Part="1"
-F 0 "D10" V 4889 3632 50  0000 R CNN
+F 0 "D12" V 4889 3632 50  0000 R CNN
 F 1 "LED" V 4798 3632 50  0000 R CNN
 F 2 "LED_SMD:LED_1206_3216Metric" H 4850 3750 50  0001 C CNN
@@
 AR Path="/610A0B30/6107B2B1" Ref="R7"  Part="1"
 AR Path="/610C441E/6107B2B1" Ref="R9"  Part="1"
-F 0 "R7" H 4920 4196 50  0000 L CNN
+F 0 "R9" H 4920 4196 50  0000 L CNN
 F 1 "1k" H 4920 4105 50  0000 L CNN
 F 2 "Resistor_SMD:R_1206_3216Metric" V 4780 4150 50  0001 C CNN

Commit message: Several changes
Usando stock de http://tienda.ityt.com.ar/
Parts:
- D8: value 1N4007 -> M7; footprint Diode_THT:D_DO-41_SOD81_P7.62mm_Horizontal -> Diode_SMD:D_SMA_Handsoldering; manf# 1N4007G -> M7
Changed lines of the file:
@@
 $Descr A4 11693 8268
 encoding utf-8
-Sheet 5 19
+Sheet 5 18
 Title "Relay Output"
 Date "2021-06-10"
@@
 AR Path="/610C441E/61070A4D" Ref="D13"  Part="1"
 F 0 "D13" V 5500 3750 50  0000 L CNN
-F 1 "1N4007" V 5600 3550 50  0000 L CNN
-F 2 "Diode_THT:D_DO-41_SOD81_P7.62mm_Horizontal" H 5550 3775 50  0001 C CNN
-F 3 "https://media.digikey.com/pdf/Data%20Sheets/NextGen%20Components%20PDFs/DO41N4007GA10A.pdf" H 5550 3950 50  0001 C CNN
-F 4 "1N4007G" H 5550 3950 50  0001 C CNN "manf#"
+F 1 "M7" V 5600 3750 50  0000 L CNN
+F 2 "Diode_SMD:D_SMA_Handsoldering" H 5550 3775 50  0001 C CNN
+F 3 "https://www.vtrons.com/images/DIODE%20M7.pdf" H 5550 3950 50  0001 C CNN
+F 4 "M7" H 5550 3950 50  0001 C CNN "manf#"
 	1    5550 3950
 	0    1    1    0
