File: psu.sch (KiCad schematic (older format))
At the start: 27 parts, among them U7 LM2596S-3.3, U7A1 ALT, U9 LM7805

Commit message: more footprints & 3d models
Parts:
- removed C10A1, C11A1, C12A1, C5A1, C6A1, C8A1, C9A1: ALT, Capacitor_THT:CP_Radial_D10.0mm_P3.80mm, symbol Device:CP
- removed L1A1: ALT, Inductor_THT:L_Radial_D12.0mm_P5.00mm_Fastron_11P, symbol Device:L
- removed U7A1: ALT, Package_TO_SOT_THT:TO-220-5_Vertical, symbol Regulator_Switching:LM2596S-3.3
- C10, C11, C12, C5, C6, C8, C9: footprint Capacitor_SMD:CP_Elec_10x10 -> libs:CAP_10x10_SMD_THT
- L1: footprint Inductor_SMD:L_12x12mm_H8mm -> libs:L_12x12mm_H8mm
- RV1: footprint Resistor_SMD:R_1206_3216Metric_Pad1.30x1.75mm_HandSolder -> Potentiometer_THT:Potentiometer_Bourns_3296W_Vertical
- U7: footprint Package_TO_SOT_SMD:TO-263-5_TabPin3 -> libs:TO-263-5_TabPin3
Other:
- note removed: "*Duplicated for dual footprint."

Commit message: Several changes
Usando stock de http://tienda.ityt.com.ar/
Parts:
- removed D7A1: ALT, Diode_THT:D_DO-201_P12.70mm_Horizontal, symbol Diode:1N5822
- removed U9: LM7805, Package_TO_SOT_THT:TO-220-3_Vertical, symbol Regulator_Linear:L7805
- added U9: AMS1117-5.0, Package_TO_SOT_SMD:SOT-223-3_TabPin2, symbol Regulator_Linear:AMS1117-5.0
Connections:
- net GND: now also U9.1 (GND)
- net VIN: now also U9.3 (VI)
- net VOUT_5V: now also U9.2 (VO)
Other:
- note removed: "*Duplicated for dual footprints."
- moved on the sheet: C10, C11, C12, C8, C9, JP1, L1, R17, RV1
