File: kicad.kicad_pcb (KiCad board)
At the start: 2 copper layers, 114 parts, among them J1 Screw_Terminal_01x02, J10 Conn_01x06, J11 ICSP, J2 Screw_Terminal_01x03, J3 Screw_Terminal_01x03, J4 Conn_01x05, J5 Screw_Terminal_01x03, J6 USB_B, J7 Conn_01x03, J8 Conn_01x03, J9 Conn_01x03, K1 RELAY, K2 RELAY, K3 RELAY, Q1 BC817, Q2 BC817, Q3 BC817, Q4 BC817, Q5 BC817, Q6 BC817, Q7 IRLML2502, SW1 SW_Push, SW2 SW_Push, U1 CH340G, U10 PC817XI, U11 DS1233A-10, U2 ACS759, U3 ACS712, U4 PC817XI, U5 PC817XI, U6 ESP32, U7 LM2596S-3.3, U8 PC817XI, U9 AMS1117-5.0, Y1 12MHz

Commit message: Closes #29
Parts:
- removed C1, C14, C15, C16, C18, C19, C20, C21, C4, C7: 100nF, Capacitor_SMD:C_1206_3216Metric_Pad1.33x1.80mm_HandSolder
- removed C10, C11, C12, C5, C6, C8, C9: 470uF, libs:CAP_10x10_SMD_THT
- removed C13: 100uF, Capacitor_THT:CP_Radial_D6.3mm_P2.50mm
- removed C17: 1nF, Capacitor_SMD:C_1206_3216Metric_Pad1.33x1.80mm_HandSolder
- removed C2, C3: 22pF, Capacitor_SMD:C_1206_3216Metric_Pad1.33x1.80mm_HandSolder
- removed D1, D2, D7: SS14, Diode_SMD:D_SMA_Handsoldering
- removed D10, D12, D5, D6: LED, LED_SMD:LED_1206_3216Metric
- removed D11, D13, D8: M7, Diode_SMD:D_SMA_Handsoldering
- removed D14, D15, D16, D9: BAT54S, Package_TO_SOT_SMD:SOT-23
- removed H1, H2: MountingHole_Pad, MountingHole:MountingHole_4mm_Pad_Via
- removed J1: Screw_Terminal_01x02, libs:TerminalBlock_bornier-2_P5.08mm
- removed J10: Conn_01x06, Connector_Molex:Molex_KK-254_AE-6410-06A_1x06_P2.54mm_Vertical
- removed J11: ICSP, Connector_PinSocket_2.54mm:PinSocket_1x06_P2.54mm_Vertical
- removed J2, J3, J5: Screw_Terminal_01x03, libs:TerminalBlock_bornier-3_P5.08mm
- removed J4: Conn_01x05, Connector_Molex:Molex_KK-254_AE-6410-05A_1x05_P2.54mm_Vertical
- removed J6: USB_B, libs:USB-B-VERTICAL-SMD&THT
- removed J7, J8, J9: Conn_01x03, Connector_Molex:Molex_KK-254_AE-6410-03A_1x03_P2.54mm_Vertical
- removed JP1: SolderJumper_2_Open, Jumper:SolderJumper-2_P1.3mm_Open_RoundedPad1.0x1.5mm
- removed JP2: SolderJumper_3_Bridged12, Jumper:SolderJumper-3_P1.3mm_Open_RoundedPad1.0x1.5mm_NumberLabels
- removed JP3, JP4, JP5: SolderJumper_2_Bridged, Jumper:SolderJumper-2_P1.3mm_Open_RoundedPad1.0x1.5mm
- removed K1, K2, K3: RELAY, Relay_THT:Relay_SPDT_SANYOU_SRD_Series_Form_C
- removed L1: 68uH, libs:L_12x12mm_H8mm
- removed Q1, Q2, Q3, Q4, Q5, Q6: BC817, Package_TO_SOT_SMD:SOT-23
- removed Q7: IRLML2502, Package_TO_SOT_SMD:SOT-23
- removed R1, R11, R12, R13, R14, R2, R28, R31, R33, R35: 10k, Resistor_SMD:R_1206_3216Metric
- removed R10, R15, R16, R18, R19, R21, R22, R23, R24, R25, R26, R27, R3, R30, R32, R34, R4, R7, R8, R9: 1k, Resistor_SMD:R_1206_3216Metric
- removed R17: 330, Resistor_SMD:R_1206_3216Metric
- removed R20: 2k, Resistor_SMD:R_1206_3216Metric
- removed R29: 100, Resistor_SMD:R_1206_3216Metric
- removed R5: 22k, Resistor_SMD:R_1206_3216Metric
- removed R6: 5k6, Resistor_SMD:R_1206_3216Metric
- removed RV1: 10k, Potentiometer_THT:Potentiometer_Bourns_3296W_Vertical
- removed SW1, SW2: SW_Push, Button_Switch_THT:SW_PUSH_6mm
- removed U1: CH340G, Package_SO:SOIC-16_3.9x9.9mm_P1.27mm
- removed U10, U4, U5, U8: PC817XI, Package_DIP:SMDIP-4_W9.53mm
- removed U11: DS1233A-10, Package_TO_SOT_THT:TO-92
- removed U2: ACS759, libs:Allegro_CB_PFF
- removed U3: ACS712, Package_SO:SOIC-8_3.9x4.9mm_P1.27mm
- removed U6: ESP32, esp32-wroom-roover:ESP32-WROOM-WROVER-NC
- removed U7: LM2596S-3.3, libs:TO-263-5_TabPin3
- removed U9: AMS1117-5.0, Package_TO_SOT_SMD:SOT-223-3_TabPin2
- removed Y1: 12MHz, Crystal:Crystal_HC49-4H_Vertical

Commit message: routeo fase 1
Parts:
- added C1: 100nF, Capacitor_SMD:C_1206_3216Metric_Pad1.33x1.80mm_HandSolder, F.Cu at (123.2, 59.7)
- added C10: 100nF, Capacitor_SMD:C_1206_3216Metric_Pad1.33x1.80mm_HandSolder, F.Cu at (148.6, 94.0)
- added C11: 100nF, Capacitor_SMD:C_1206_3216Metric_Pad1.33x1.80mm_HandSolder, F.Cu at (137.2, 98.7)
- added C12: 100nF, Capacitor_SMD:C_1206_3216Metric_Pad1.33x1.80mm_HandSolder, F.Cu at (145.4, 90.8)
- added C13: 1nF, Capacitor_SMD:C_1206_3216Metric_Pad1.33x1.80mm_HandSolder, F.Cu at (147.3, 98.7)
- added C2: 1uF, Capacitor_SMD:C_1206_3216Metric_Pad1.33x1.80mm_HandSolder, F.Cu at (120.7, 59.7)
- added C3: 100nF, Capacitor_SMD:C_1206_3216Metric_Pad1.33x1.80mm_HandSolder, B.Cu at (169.0, 59.0)
- added C4: 100nF, Capacitor_SMD:C_1206_3216Metric_Pad1.33x1.80mm_HandSolder, B.Cu at (177.0, 53.0)
- added C5: 100nF, Capacitor_SMD:C_1206_3216Metric_Pad1.33x1.80mm_HandSolder, B.Cu at (178.5, 59.0)
- added C6: 100nF, Capacitor_SMD:C_1206_3216Metric_Pad1.33x1.80mm_HandSolder, B.Cu at (167.5, 53.0)
- added C7: 470uF, libs:CAP_10x10_SMD_THT, F.Cu at (106.0, 106.5)
- added C8: 100nF, Capacitor_SMD:C_1206_3216Metric_Pad1.33x1.80mm_HandSolder, F.Cu at (106.0, 100.0)
- added C9: 470uF, libs:CAP_10x10_SMD_THT, F.Cu at (130.2, 88.9)
- added D1: SS14, Diode_SMD:D_SMA_Handsoldering, F.Cu at (97.2, 106.5)
- added D10: LED, LED_SMD:LED_1206_3216Metric, F.Cu at (94.0, 104.0)
- added D11: SS14, Diode_SMD:D_SMA_Handsoldering, F.Cu at (118.1, 100.3)
- added D12: BAT54S, Package_TO_SOT_SMD:SOT-23, B.Cu at (109.0, 100.0)
- added D13: BAT54S, Package_TO_SOT_SMD:SOT-23, F.Cu at (143.5, 86.9)
- added D2: LED, LED_SMD:LED_1206_3216Metric, F.Cu at (154.2, 80.9)
- added D3: M7, Diode_SMD:D_SMA_Handsoldering, F.Cu at (158.1, 82.8)
- added D4: LED, LED_SMD:LED_1206_3216Metric, F.Cu at (154.2, 98.7)
- added D5: M7, Diode_SMD:D_SMA_Handsoldering, F.Cu at (158.1, 100.6)
- added D6: LED, LED_SMD:LED_1206_3216Metric, F.Cu at (154.2, 63.1)
- added D7: M7, Diode_SMD:D_SMA_Handsoldering, F.Cu at (158.1, 65.0)
- added D8: BAT54S, Package_TO_SOT_SMD:SOT-23, F.Cu at (150.0, 68.0)
- added D9: BAT54S, Package_TO_SOT_SMD:SOT-23, F.Cu at (150.0, 78.0)
- added H1: MountingHole_Pad, MountingHole:MountingHole_4mm_Pad_Via, F.Cu at (127.2, 115.5)
- added H2: MountingHole_Pad, MountingHole:MountingHole_4mm_Pad_Via, F.Cu at (157.2, 115.5)
- added J1: Screw_Terminal_01x02, libs:TerminalBlock_bornier-2_P5.08mm, F.Cu at (104.0, 116.0)
- added J10: Conn_01x10, Connector_Molex:Molex_KK-254_AE-6410-10A_1x10_P2.54mm_Vertical, F.Cu at (96.0, 84.9)
- added J2: Screw_Terminal_01x03, libs:TerminalBlock_bornier-3_P5.08mm, F.Cu at (186.0, 91.1)
- added J3: Screw_Terminal_01x03, libs:TerminalBlock_bornier-3_P5.08mm, F.Cu at (186.0, 108.9)
- added J4: Screw_Terminal_01x03, libs:TerminalBlock_bornier-3_P5.08mm, F.Cu at (186.0, 73.3)
- added J5: Conn_01x03, Connector_Molex:Molex_KK-254_AE-6410-03A_1x03_P2.54mm_Vertical, F.Cu at (179.7, 116.2)
- added J6: ICSP, Connector_PinSocket_2.54mm:PinSocket_1x06_P2.54mm_Vertical, F.Cu at (104.7, 54.5)
- added J7: Conn_01x05, Connector_Molex:Molex_KK-254_AE-6410-05A_1x05_P2.54mm_Vertical, F.Cu at (149.9, 55.9)
- added J8: Conn_01x03, Connector_Molex:Molex_KK-254_AE-6410-03A_1x03_P2.54mm_Vertical, F.Cu at (165.1, 55.9)
- added J9: Conn_01x03, Connector_Molex:Molex_KK-254_AE-6410-03A_1x03_P2.54mm_Vertical, F.Cu at (174.6, 55.9)
- added JP2: SolderJumper_3_Bridged12, Jumper:SolderJumper-3_P1.3mm_Open_RoundedPad1.0x1.5mm_NumberLabels, F.Cu at (140.3, 90.8)
- added JP3: SolderJumper_2_Open, Jumper:SolderJumper-2_P1.3mm_Open_RoundedPad1.0x1.5mm, B.Cu at (100.5, 83.5)
- added K1: RELAY, Relay_THT:Relay_SPDT_SANYOU_SRD_Series_Form_C, F.Cu at (162.3, 86.0)
- added K2: RELAY, Relay_THT:Relay_SPDT_SANYOU_SRD_Series_Form_C, F.Cu at (162.3, 103.8)
- added K3: RELAY, Relay_THT:Relay_SPDT_SANYOU_SRD_Series_Form_C, F.Cu at (162.3, 68.2)
- added L1: 68uH, libs:L_12x12mm_H8mm, F.Cu at (116.2, 92.1)
- added Q1: BC817, Package_TO_SOT_SMD:SOT-23, F.Cu at (158.1, 91.1)
- added Q2: BC817, Package_TO_SOT_SMD:SOT-23, F.Cu at (158.1, 108.9)
- added Q3: BC817, Package_TO_SOT_SMD:SOT-23, F.Cu at (158.1, 73.3)
- added Q4: BC817, Package_TO_SOT_SMD:SOT-23, F.Cu at (165.1, 117.5)
- added Q5: IRLML2502, Package_TO_SOT_SMD:SOT-23, F.Cu at (170.8, 117.5)
- added R1: 22k, Resistor_SMD:R_1206_3216Metric, F.Cu at (100.0, 100.0)
- added R10: 1k, Resistor_SMD:R_1206_3216Metric, F.Cu at (153.0, 108.0)
- added R11: 1k, Resistor_SMD:R_1206_3216Metric, F.Cu at (154.2, 68.2)
- added R12: 1k, Resistor_SMD:R_1206_3216Metric, F.Cu at (154.2, 73.3)
- added R13: 1k, Resistor_SMD:R_1206_3216Metric, F.Cu at (150.0, 64.5)
- added R14: 1k, Resistor_SMD:R_1206_3216Metric, F.Cu at (150.0, 71.5)
- added R15: 1k, Resistor_SMD:R_1206_3216Metric, F.Cu at (150.0, 74.5)
- added R16: 1k, Resistor_SMD:R_1206_3216Metric, F.Cu at (150.0, 81.5)
- added R17: 1k, Resistor_SMD:R_1206_3216Metric, F.Cu at (94.0, 109.0)
- added R19: 1k, Resistor_SMD:R_1206_3216Metric, B.Cu at (103.0, 100.0)
- added R2: 5k6, Resistor_SMD:R_1206_3216Metric, F.Cu at (95.0, 100.0)
- added R20: 1k, Resistor_SMD:R_1206_3216Metric, B.Cu at (115.0, 100.0)
- added R21: 2k, Resistor_SMD:R_1206_3216Metric, F.Cu at (144.1, 98.7)
- added R22: 1k, Resistor_SMD:R_1206_3216Metric, F.Cu at (140.3, 98.7)
- added R23: 1k, Resistor_SMD:R_1206_3216Metric, F.Cu at (165.7, 114.3)
- added R24: 10k, Resistor_SMD:R_1206_3216Metric, F.Cu at (170.8, 114.3)
- added R25: 1k, Resistor_SMD:R_1206_3216Metric, F.Cu at (139.7, 87.0)
- added R26: 1k, Resistor_SMD:R_1206_3216Metric, F.Cu at (147.3, 87.0)
- added R27: 100, Resistor_SMD:R_1206_3216Metric, F.Cu at (116.0, 79.5)
- added R28: 100, Resistor_SMD:R_1206_3216Metric, F.Cu at (116.0, 76.5)
- added R29: 1k, Resistor_SMD:R_1206_3216Metric, B.Cu at (108.0, 70.0)
- added R3: 10k, Resistor_SMD:R_1206_3216Metric, F.Cu at (123.8, 107.3)
- added R30: 10k, Resistor_SMD:R_1206_3216Metric, B.Cu at (120.0, 70.0)
- added R31: 1k, Resistor_SMD:R_1206_3216Metric, B.Cu at (108.0, 67.0)
- added R32: 10k, Resistor_SMD:R_1206_3216Metric, B.Cu at (120.0, 73.0)
- added R33: 1k, Resistor_SMD:R_1206_3216Metric, B.Cu at (108.0, 64.0)
- added R34: 10k, Resistor_SMD:R_1206_3216Metric, B.Cu at (120.0, 64.0)
- added R35: 1k, Resistor_SMD:R_1206_3216Metric, B.Cu at (108.0, 60.5)
- added R36: 10k, Resistor_SMD:R_1206_3216Metric, B.Cu at (120.0, 67.0)
- added R4: 10k, Resistor_SMD:R_1206_3216Metric, F.Cu at (127.0, 107.3)
- added R5: 10k, Resistor_SMD:R_1206_3216Metric, B.Cu at (152.4, 59.7)
- added R6: 10k, Resistor_SMD:R_1206_3216Metric, B.Cu at (149.9, 59.7)
- added R7: 1k, Resistor_SMD:R_1206_3216Metric, F.Cu at (154.2, 86.0)
- added R8: 1k, Resistor_SMD:R_1206_3216Metric, F.Cu at (154.2, 91.1)
- added R9: 1k, Resistor_SMD:R_1206_3216Metric, F.Cu at (154.2, 103.8)
- added REF**: MountingHole_3.5mm_Pad, MountingHole:MountingHole_3.5mm_Pad, F.Cu at (186.3, 56.0)
- added REF**: MountingHole_3.5mm_Pad, MountingHole:MountingHole_3.5mm_Pad, F.Cu at (96.3, 116.0)
- added REF**: MountingHole_3.5mm_Pad, MountingHole:MountingHole_3.5mm_Pad, F.Cu at (186.3, 116.0)
- added REF**: MountingHole_3.5mm_Pad, MountingHole:MountingHole_3.5mm_Pad, F.Cu at (96.3, 56.0)
- added SW1: SW_Push, Button_Switch_THT:SW_PUSH_6mm, F.Cu at (114.2, 105.1)
- added SW2: SW_Push, Button_Switch_THT:SW_PUSH_6mm, F.Cu at (114.2, 114.0)
- added U1: DS1233A-10, Package_TO_SOT_THT:TO-92, F.Cu at (131.8, 108.6)
- added U10: PC817XI, Package_DIP:SMDIP-4_W9.53mm, F.Cu at (120.0, 65.5)
- added U11: PC817XI, Package_DIP:SMDIP-4_W9.53mm, F.Cu at (107.0, 65.5)
- added U12: PC817XI, Package_DIP:SMDIP-4_W9.53mm, F.Cu at (107.0, 59.5)
- added U2: ESP32, esp32-wroom-roover:ESP32-WROOM-WROVER-NC, F.Cu at (136.5, 66.7)
- added U3: LM2596S-3.3, libs:TO-263-5_TabPin3, F.Cu at (100.3, 93.0)
- added U4: AMS1117-5.0, Package_TO_SOT_SMD:SOT-223-3_TabPin2, F.Cu at (128.3, 100.2)
- added U5: ACS759, libs:Allegro_CB_PFF, F.Cu at (144.1, 93.6)
- added U6: ACS712, Package_SO:SOIC-8_3.9x4.9mm_P1.27mm, F.Cu at (142.2, 105.4)
- added U7: PC817XI, Package_DIP:SMDIP-4_W9.53mm, F.Cu at (107.0, 80.5)
- added U8: PC817XI, Package_DIP:SMDIP-4_W9.53mm, F.Cu at (107.0, 75.0)
- added U9: PC817XI, Package_DIP:SMDIP-4_W9.53mm, F.Cu at (120.0, 71.5)
Routing:
- net /Relay 3/COM: track 0.00 -> 47.5 mm
- net /Relay 2/COM: track 0.00 -> 47.5 mm
- net /Relay 1/COM: track 0.00 -> 47.5 mm
- net +3V3: track 0.00 -> 37.1 mm
- net +12V: track 0.00 -> 35.1 mm
- net /Relay 3/NO: track 0.00 -> 20.0 mm
- net /Relay 2/NO: track 0.00 -> 20.0 mm
- net /Relay 1/NO: track 0.00 -> 20.0 mm
- net GPIO0: track 0.00 -> 19.9 mm
- net /Relay 3/NC: track 0.00 -> 19.8 mm
- net /Relay 2/NC: track 0.00 -> 19.8 mm
- net /Relay 1/NC: track 0.00 -> 19.8 mm
- net RESET: track 0.00 -> 19.4 mm
- net Net-(D11-Pad1): track 0.00 -> 16.0 mm
- net Net-(D7-Pad2): track 0.00 -> 15.8 mm
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- added copper zone on F.Cu, net +12V
- added copper zone on B.Cu, net +5V
- added copper zone on F.Cu, net +5V
- added copper zone on B.Cu, net /Current Sensor/IP+
- added copper zone on F.Cu, net /Current Sensor/IP+
- added copper zone on B.Cu, net /Current Sensor/IP-
- added copper zone on F.Cu, net /Current Sensor/IP-
- added copper zone on B.Cu, net GND
- added copper zone on F.Cu, net GND
- added copper zone on F.Cu, net Net-(D11-Pad1)
Other:
- board outline added: 100 x 70 mm
- net class Default removed
- board text added: "PROG"
- board text added: "RESET"

Commit message: fix bugardo
Connections:
- J10 pad 1: +12V -> GND
Changed lines of the file:
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@@
     (fp_line (start 24.13 2.88) (end 24.13 -2.92) (layer "F.Fab") (width 0.1))
     (pad "1" thru_hole roundrect (at 0 0 90) (size 1.74 2.19) (drill 1.19) (layers *.Cu *.Mask) (roundrect_rratio 0.143678)
-      (net 3 "+12V") (pinfunction "Pin_1") (pintype "passive"))
+      (net 2 "GND") (pinfunction "Pin_1") (pintype "passive"))
     (pad "2" thru_hole oval (at 2.54 0 90) (size 1.74 2.19) (drill 1.19) (layers *.Cu *.Mask)
       (net 38 "/Opto I/O/input-0/A") (pinfunction "Pin_2") (pintype "passive"))
@@
   (via (at 110 88) (size 0.8) (drill 0.4) (layers "F.Cu" "B.Cu") (free) (net 2))
   (via (at 94.742 96.52) (size 0.8) (drill 0.4) (layers "F.Cu" "B.Cu") (free) (net 2))
+  (segment locked (start 164.21 62.27) (end 158.335 62.27) (width 1) (layer "F.Cu") (net 3))
   (segment locked (start 158.335 97.83) (end 158.06 98.105) (width 1) (layer "F.Cu") (net 3))
-  (segment locked (start 158.335 62.27) (end 158.06 62.545) (width 1) (layer "F.Cu") (net 3))
-  (segment locked (start 158.335 80.05) (end 158.06 80.325) (width 1) (layer "F.Cu") (net 3))
+  (segment locked (start 157.255 61.74) (end 158.06 62.545) (width 1) (layer "F.Cu") (net 3))
   (segment locked (start 154.25 97.3) (end 157.255 97.3) (width 1) (layer "F.Cu") (net 3))
-  (segment locked (start 154.25 61.74) (end 157.255 61.74) (width 1) (layer "F.Cu") (net 3))
-  (segment locked (start 154.25 79.52) (end 157.255 79.52) (width 1) (layer "F.Cu") (net 3))
   (segment (start 94 102.6) (end 95.996 102.6) (width 1) (layer "F.Cu") (net 3))
+  (segment locked (start 154.25 79.52) (end 157.255 79.52) (width 1) (layer "F.Cu") (net 3))
+  (segment locked (start 157.255 79.52) (end 158.06 80.325) (width 1) (layer "F.Cu") (net 3))
+  (segment locked (start 154.25 61.74) (end 157.255 61.74) (width 1) (layer "F.Cu") (net 3))
   (segment locked (start 164.21 97.83) (end 158.335 97.83) (width 1) (layer "F.Cu") (net 3))
-  (segment locked (start 164.21 62.27) (end 158.335 62.27) (width 1) (layer "F.Cu") (net 3))
   (segment locked (start 164.21 80.05) (end 158.335 80.05) (width 1) (layer "F.Cu") (net 3))
   (segment (start 95.996 102.6) (end 97.155 103.759) (width 1) (layer "F.Cu") (net 3))
+  (segment locked (start 158.335 80.05) (end 158.06 80.325) (width 1) (layer "F.Cu") (net 3))
+  (segment locked (start 158.335 62.27) (end 158.06 62.545) (width 1) (layer "F.Cu") (net 3))
   (segment locked (start 157.255 97.3) (end 158.06 98.105) (width 1) (layer "F.Cu") (net 3))
-  (segment locked (start 157.255 61.74) (end 158.06 62.545) (width 1) (layer "F.Cu") (net 3))
-  (segment locked (start 157.255 79.52) (end 158.06 80.325) (width 1) (layer "F.Cu") (net 3))
   (segment (start 97.155 103.759) (end 97.155 104) (width 1) (layer "F.Cu") (net 3))
   (segment (start 137.15 100.2275) (end 137.15 100.955) (width 1) (layer "F.Cu") (net 4))
@@
   (segment (start 185.912 80.899) (end 177.292 80.899) (width 2) (layer "B.Cu") (net 15))
   (segment (start 177.292 80.899) (end 176.372 79.979) (width 2) (layer "B.Cu") (net 15))
-  (segment locked (start 177.38 108.86) (end 176.41 109.83) (width 2) (layer "F.Cu") (net 16))
   (segment locked (start 186 108.86) (end 177.38 108.86) (width 2) (layer "F.Cu") (net 16))
+  (segment locked (start 177.38 108.86) (end 176.41 109.83) (width 2) (layer "F.Cu") (net 16))
   (segment (start 177.292 108.839) (end 176.322 109.809) (width 2) (layer "B.Cu") (net 16))
   (segment (start 185.912 108.839) (end 177.292 108.839) (width 2) (layer "B.Cu") (net 16))
@@
   (segment (start 149.86 58.2275) (end 149.86 55.9) (width 0.25) (layer "B.Cu") (net 19))
   (segment (start 152.4 58.2275) (end 152.4 55.9) (width 0.25) (layer "B.Cu") (net 20))
-  (segment locked (start 177.38 73.3) (end 176.41 74.27) (width 2) (layer "F.Cu") (net 21))
   (segment locked (start 186 73.3) (end 177.38 73.3) (width 2) (layer "F.Cu") (net 21))
+  (segment locked (start 177.38 73.3) (end 176.41 74.27) (width 2) (layer "F.Cu") (net 21))
   (segment (start 177.292 73.279) (end 176.322 74.249) (width 2) (layer "B.Cu") (net 21))
   (segment (start 185.912 73.279) (end 177.292 73.279) (width 2) (layer "B.Cu") (net 21))
@@
   (segment locked (start 154.25 89.6175) (end 154.7625 90.13) (width 0.25) (layer "F.Cu") (net 40))
   (segment locked (start 154.7625 90.13) (end 157.1225 90.13) (width 0.25) (layer "F.Cu") (net 40))
-  (segment locked (start 154.25 71.8375) (end 154.7625 72.35) (width 0.25) (layer "F.Cu") (net 42))
   (segment locked (start 154.7625 72.35) (end 157.1225 72.35) (width 0.25) (layer "F.Cu") (net 42))
+  (segment locked (start 154.25 71.8375) (end 154.7625 72.35) (width 0.25) (layer "F.Cu") (net 42))
   (segment (start 141.635 90.805) (end 141.635 92.27) (width 0.25) (layer "F.Cu") (net 59))
   (segment (start 141.635 92.27) (end 140.32 93.585) (width 0.25) (layer "F.Cu") (net 59))
@@
   (segment locked (start 154.25 87.4625) (end 155.863572 87.4625) (width 0.25) (layer "F.Cu") (net 62))
   (segment locked (start 154.25 100.1) (end 154.25 102.3175) (width 0.25) (layer "F.Cu") (net 63))
-  (segment locked (start 158.06 105.685) (end 158.9975 106.6225) (width 0.25) (layer "F.Cu") (net 64))
+  (segment locked (start 154.25 105.2425) (end 155.863572 105.2425) (width 0.25) (layer "F.Cu") (net 64))
+  (segment locked (start 155.863572 105.2425) (end 156.306072 105.685) (width 0.25) (layer "F.Cu") (net 64))
+  (segment locked (start 158.06 103.105) (end 158.06 105.685) (width 0.25) (layer "F.Cu") (net 64))
   (segment locked (start 156.306072 105.685) (end 158.06 105.685) (width 0.25) (layer "F.Cu") (net 64))
-  (segment locked (start 161.87 108.86) (end 158.9975 108.86) (width 0.25) (layer "F.Cu") (net 64))
   (segment locked (start 158.9975 106.6225) (end 158.9975 108.86) (width 0.25) (layer "F.Cu") (net 64))
+  (segment locked (start 161.87 108.86) (end 158.9975 108.86) (width 0.25) (layer "F.Cu") (net 64))
   (segment locked (start 164.21 109.83) (end 162.84 109.83) (width 0.25) (layer "F.Cu") (net 64))
-  (segment locked (start 158.06 103.105) (end 158.06 105.685) (width 0.25) (layer "F.Cu") (net 64))
+  (segment locked (start 158.06 105.685) (end 158.9975 106.6225) (width 0.25) (layer "F.Cu") (net 64))
   (segment locked (start 162.84 109.83) (end 161.87 108.86) (width 0.25) (layer "F.Cu") (net 64))
-  (segment locked (start 155.863572 105.2425) (end 156.306072 105.685) (width 0.25) (layer "F.Cu") (net 64))
-  (segment locked (start 154.25 105.2425) (end 155.863572 105.2425) (width 0.25) (layer "F.Cu") (net 64))
-  (segment locked (start 158.06 70.125) (end 158.9975 71.0625) (width 0.25) (layer "F.Cu") (net 65))
-  (segment locked (start 156.306072 70.125) (end 158.06 70.125) (width 0.25) (layer "F.Cu") (net 65))
   (segment locked (start 161.87 73.3) (end 158.9975 73.3) (width 0.25) (layer "F.Cu") (net 65))
-  (segment locked (start 158.9975 71.0625) (end 158.9975 73.3) (width 0.25) (layer "F.Cu") (net 65))
-  (segment locked (start 164.21 74.27) (end 162.84 74.27) (width 0.25) (layer "F.Cu") (net 65))
-  (segment locked (start 158.06 67.545) (end 158.06 70.125) (width 0.25) (layer "F.Cu") (net 65))
+  (segment locked (start 156.306072 70.125) (end 158.06 70.125) (width 0.25) (layer "F.Cu") (net 65))
   (segment locked (start 162.84 74.27) (end 161.87 73.3) (width 0.25) (layer "F.Cu") (net 65))
   (segment locked (start 155.863572 69.6825) (end 156.306072 70.125) (width 0.25) (layer "F.Cu") (net 65))
+  (segment locked (start 164.21 74.27) (end 162.84 74.27) (width 0.25) (layer "F.Cu") (net 65))
+  (segment locked (start 158.06 70.125) (end 158.9975 71.0625) (width 0.25) (layer "F.Cu") (net 65))
   (segment locked (start 154.25 69.6825) (end 155.863572 69.6825) (width 0.25) (layer "F.Cu") (net 65))
+  (segment locked (start 158.06 67.545) (end 158.06 70.125) (width 0.25) (layer "F.Cu") (net 65))
+  (segment locked (start 158.9975 71.0625) (end 158.9975 73.3) (width 0.25) (layer "F.Cu") (net 65))
   (segment (start 115.61 100.33) (end 115.61 98.084) (width 1) (layer "F.Cu") (net 67))
   (segment (start 106.105 94.7) (end 111.21 94.7) (width 1) (layer "F.Cu") (net 67))
@@
     (min_thickness 0.254)
     (keepout (tracks not_allowed) (vias allowed) (pads allowed ) (copperpour not_allowed) (footprints allowed))
-    (fill (thermal_gap 0.508) (thermal_bridge_width 0.508) (smoothing fillet) (radius 1))
+    (fill (thermal_gap 0.508) (thermal_bridge_width 0.508))
     (polygon
       (pts
@@
         (xy 126.492 104.394)
         (xy 126.492 101.092)
-        (xy 126.492 101.092)
-        (xy 126.492 99.314)
         (xy 126.492 99.314)
         (xy 126.492 94.234)
@@
         (xy 126.492 104.394)
         (xy 126.492 101.092)
-        (xy 126.492 101.092)
-        (xy 126.492 99.314)
         (xy 126.492 99.314)
         (xy 126.492 94.234)
