File: kicad.kicad_pcb (KiCad board)
At the start: 2 copper layers, 100 x 70 mm, 102 parts, among them J1 Screw_Terminal_01x02, J10 Conn_01x10, J2 Screw_Terminal_01x03, J3 Screw_Terminal_01x03, J4 Screw_Terminal_01x03, J5 Conn_01x03, J6 ICSP, J7 Conn_01x05, J8 Conn_01x03, J9 Conn_01x03, K1 RELAY, K2 RELAY, K3 RELAY, Q1 BC817, Q2 BC817, Q3 BC817, Q4 BC817, Q5 IRLML2502, SW1 SW_Push, SW2 SW_Push, U1 DS1233A-10, U10 PC817XI, U11 PC817XI, U12 PC817XI, U2 ESP32, U3 LM2596S-3.3, U4 AMS1117-5.0, U5 ACS759, U6 ACS712, U7 PC817XI, U8 PC817XI, U9 PC817XI

Commit message: fix bugardo - routeos principales
Routing:
- net +12V: track 35.1 -> 152.1 mm
- net +5V: track 10.5 -> 55.4 mm
- net +3V3: track 37.1 -> 72.2 mm
- net /Opto I/O/input-1/K: track 0.00 -> 22.9 mm
- net /Opto I/O/input-0/K: track 0.00 -> 20.5 mm
- net SDA: track 2.33 -> 15.2 mm
- net SCL: track 2.33 -> 11.3 mm
- net Net-(D8-Pad3): track 0.00 -> 8.63 mm
- net Net-(D9-Pad3): track 0.00 -> 8.43 mm
- net /Opto I/O/input-2/K: track 0.00 -> 7.11 mm
- net /Opto I/O/output-1/E: track 0.00 -> 7.01 mm
- net /Opto I/O/output-1/C: track 0.00 -> 7.01 mm
- net /Opto I/O/output-0/E: track 0.00 -> 6.84 mm
- net /Opto I/O/output-0/C: track 0.00 -> 6.84 mm
- net /Opto I/O/input-3/K: track 0.00 -> 6.75 mm
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