File: kicad.kicad_sch (KiCad schematic)
At the start: 22 parts, among them J1 Screw_Terminal_01x02, J2 Screw_Terminal_01x03, J3 Screw_Terminal_01x03, J4 Screw_Terminal_01x03, J5 Conn_01x03, J6 ICSP, J7 Conn_01x05, SW1 SW_Push, SW2 SW_Push, U1 DS1233A-10

Commit message: fix bugardo
Parts:
- U2: value (none) -> ESP32; footprint (none) -> esp32-wroom-roover:ESP32-WROOM-WROVER-NC
Changed lines of the file:
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@@
     (in_bom yes) (on_board yes)
     (property "Reference" "U2" (id 0) (at 238.76 105.41 0))
-    (property "Value" "" (id 1) (at 259.08 105.41 0))
-    (property "Footprint" "" (id 2) (at 250.19 177.8 0)
+    (property "Value" "ESP32" (id 1) (at 259.08 105.41 0))
+    (property "Footprint" "esp32-wroom-roover:ESP32-WROOM-WROVER-NC" (id 2) (at 250.19 177.8 0)
       (effects (font (size 1.27 1.27)) hide)
     )
@@
       (reference "#PWR077") (unit 1) (value "+3V3") (footprint "")
     )
+    (path "/00000000-0000-0000-0000-00006174a55c/add4f416-1cd8-4b85-b16a-fdd542b7564e"
+      (reference "#PWR?") (unit 1) (value "GND") (footprint "")
+    )
     (path "/00000000-0000-0000-0000-000060ca50a5"
